Commit message: Fix: Remove duplicate world link definition to resolve robot_state_publisher root link error
The URDF parser requires exactly one root link (a link with no parent).
Previously, both 'world' and 'base_link' were root links, causing the error:
"Failed to find root link: Two root links found: [base_link] and [world]"

The 'world' frame is automatically managed by robot_state_publisher and doesn't
need to be explicitly defined in the URDF.

File: src/lebai_gazebo/urdf/lm3_gazebo.xacro (robot description, xacro)
@@ -12,11 +12,11 @@
 ========================================================================= -->
 <robot xmlns:xacro="http://www.ros.org/wiki/xacro" name="lebai_lm3">
-  <!-- 世界根 -->
-  <link name="world"/>
   <!-- 复用已有机械臂宏。注意: lm3_macro.xacro 末尾已经自带
        <xacro:lebai_lm3 prefix="lebai_"/> 的实例化, 这里只 include, 不要再实例化,
        否则链接/关节重名报错。 -->
   <xacro:include filename="$(find lebai_lm3_support)/urdf/lm3_macro.xacro"/>
-  <!-- 底座固定到世界, 抬到桌面高度(与 world 文件里的桌子一致) -->
+  <!-- 底座固定到世界, 抬到桌面高度(与 world 文件里的桌子一致)
+       注: world 是 robot_state_publisher 自动创建的虚拟根链接,
+           URDF 中不需要显式定义 -->
   <joint name="world_to_base" type="fixed">
     <parent link="world"/>

Commit message: Fix: Remove world_to_base joint to resolve robot_state_publisher parsing error
The robot_state_publisher requires URDF to have a single root link that exists
when the URDF is parsed. The 'world' link is not a real link but a virtual 
frame created dynamically by robot_state_publisher.

By removing the world_to_base joint, lebai_base_link becomes the root link,
and robot_state_publisher will properly create the TF tree. The robot's
position in Gazebo is controlled via the spawn_entity node or the world file.

File: src/lebai_gazebo/urdf/lm3_gazebo.xacro (robot description, xacro)
@@ -3,5 +3,4 @@
   lm3_gazebo.xacro — Gazebo(Classic 11) 仿真用的 LM3 机械臂描述。
   在原有 lm3_macro.xacro 基础上补充 Gazebo 仿真所需:
-    - 把机械臂底座固定到 world(桌面臂);
     - ros2_control(GazeboSystem) + gazebo_ros2_control 插件, 让臂在仿真里可被控制
       (控制器名 lebai_trajectory_controller, 与 MoveIt 的 lm3_controllers.yaml 一致);
@@ -10,4 +9,5 @@
   注意: 相机安装位置(tool0->camera 的 origin)和内参需按实际手眼标定微调;
         这是仿真脚手架, 真机上的精确数值请以标定为准。
+        Gazebo 中机械臂的高度由 world 文件中的模型位置控制, 而不是 URDF.
 ========================================================================= -->
 <robot xmlns:xacro="http://www.ros.org/wiki/xacro" name="lebai_lm3">
@@ -16,12 +16,4 @@
        否则链接/关节重名报错。 -->
   <xacro:include filename="$(find lebai_lm3_support)/urdf/lm3_macro.xacro"/>
-  <!-- 底座固定到世界, 抬到桌面高度(与 world 文件里的桌子一致)
-       注: world 是 robot_state_publisher 自动创建的虚拟根链接,
-           URDF 中不需要显式定义 -->
-  <joint name="world_to_base" type="fixed">
-    <parent link="world"/>
-    <child link="lebai_base_link"/>
-    <origin xyz="0 0 1.015" rpy="0 0 0"/>
-  </joint>
   <!-- ===================== eye-in-hand 相机 ===================== -->
   <link name="camera_arm_link">
